Commit message: added some files/folders
URDF and launch files, need stl files for frame and wheels to create meshes for the robot urdf file. Currently not loading inside the igvc world until then

File: src/lane_follower/urdf/turbo_blue.urdf (robot description, URDF)
Before this commit: robot igvc_robot, 5 links, 4 joints
Links:
- removed link chassis
- removed link front_left_wheel
- removed link front_right_wheel
- removed link rear_left_wheel
- removed link rear_right_wheel
- added link base_link; collision box size=0.4064 0.9652 0.3556; visual box size=0.4064 0.9652 0.3556
- added link camera_mount
- added link caster_swivel
- added link caster_wheel
- added link left_wheel
- added link lidar_mount
- added link right_wheel
Joints:
- removed joint front_left_wheel_joint
- removed joint front_right_wheel_joint
- removed joint rear_left_wheel_joint
- removed joint rear_right_wheel_joint
- added joint camera_mount_joint: type fixed, parent base_link, child camera_mount, origin xyz=0 0 0.4556 rpy=0 0 0
- added joint caster_swivel_joint: type revolute, parent base_link, child caster_swivel, origin xyz=-0.3048 0 0 rpy=0 0 0, axis 0 0 1, limit lower=-3.14 upper=3.14 effort=0.1 velocity=1.0
- added joint caster_wheel_spin: type continuous, parent caster_swivel, child caster_wheel, origin xyz=0 -0.08202 -0.0508 rpy=0 0 0, axis 0 1 0
- added joint left_wheel_joint: type continuous, parent base_link, child left_wheel, origin xyz=0 0.2032 0 rpy=0 0 0, axis 0 1 0
- added joint lidar_mount_joint: type fixed, parent base_link, child lidar_mount, origin xyz=0 0 0.4756 rpy=0 0 0
- added joint right_wheel_joint: type continuous, parent base_link, child right_wheel, origin xyz=0 -0.2032 0 rpy=0 0 0, axis 0 1 0
